File: kicad/c_holes.sch (KiCad schematic (older format))
At the start: 0 parts

Commit message: with fastrax gps, lsm303 footprint, ad7193
Parts:
- added C2, C3, C4, C5: C, symbol C
- added P1: CONN_4, symbol CONN_4
- added U3: P8X32A-LQFP, symbol P8X32A-LQFP
- added U4: LSM303DLHC, ~, symbol LSM303DLHC
- added U5: CAT24C256, symbol CAT24C256
- added U6: U501-GPS, symbol U501-GPS
- added X1: CRYSTAL, symbol CRYSTAL
Connections:
- new net: U3.28 (XI), X1.2
- new net: U3.29 (X0), X1.1
- new net: U3.35 (P28), U5.6 (SCL)
- new net: U3.36 (P29), U5.5 (SDA)
- new net: P1.4 (P4), U3.37 (P30)
- new net: P1.3 (P3), U3.38 (P31)
- new net: P1.1 (P1), U3.7 (RESn)
- new net PPSGPS: U3.20 (P17), U6.6 (PPB)
- new net RXDGPS: U3.22 (P19), U6.1 (RXD)
- new net SCLACC: U3.13 (P12), U4.2 (SCL)
- new net SDAACC: U3.14 (P13), U4.3 (SDA)
- new net TXDGPS: U3.21 (P18), U6.2 (TXD)
- new net VDD: C2.1, C3.1, C4.1, C5.1, U3.18 (VDD), U3.30 (VDD), U3.40 (VDD), U3.8 (VDD), U4.14 (Vdd), U5.8 (VCC), U6.4 (VDD), U6.5 (VDD_B)
- new net VSS: C2.2, C3.2, C4.2, C5.2, P1.2 (P2), U3.17 (VSS), U3.27 (VSS), U3.39 (VSS), U3.5 (VSS), U3.6 (BOEn), U4.7 (GND), U5.1 (A0), U5.2 (A1), U5.3 (A2), U5.4 (GND), U5.7 (WP), U6.3 (GND)
